Commit message: added RPLidar A1 edits.

File: description/lidar_orig.xacro (robot description, xacro)
@@ -1,35 +1,24 @@
 <?xml version="1.0"?>
-<robot xmlns:xacro="http://www.ros.org/wiki/xacro">
-  <!-- Macro parameters: parent link, XYZ offset, RPY offset -->
-  <xacro:macro name="rplidar_a1" params="parent *origin">
+<robot xmlns:xacro="http://www.ros.org/wiki/xacro" >
     <joint name="laser_joint" type="fixed">
-      <xacro:insert_block name="origin"/>
-      <parent link="${parent}"/>
-      <child link="laser_frame"/>
+        <parent link="chassis"/>
+        <child link="laser_frame"/>
+        <origin xyz="0.1 0 0.175" rpy="0 0 0"/>
     </joint>
     <link name="laser_frame">
-      <visual>
-        <geometry>
-          <!-- A1 approximate dimensions: 98.5mm diameter, 60mm height -->
-          <cylinder radius="0.0493" length="0.060"/>
-        </geometry>
-        <material name="lidar_red">
-          <color rgba="0.8 0.0 0.0 1.0"/>
-        </material>
-      </visual>
-      <collision>
-        <geometry>
-          <cylinder radius="0.0493" length="0.060"/>
-        </geometry>
-      </collision>
-      <inertial>
-        <!-- RPLIDAR A1M8 mass: ~170g -->
-        <mass value="0.170"/>
-        <!-- Solid cylinder: Ixx = Iyy = m(3r² + h²)/12, Izz = mr²/2 -->
-        <inertia
-          ixx="0.000214" ixy="0.0" ixz="0.0"
-          iyy="0.000214" iyz="0.0"
-          izz="0.000205"/>
-      </inertial>
+        <visual>
+            <geometry>
+                <cylinder radius="0.05" length="0.04"/>
+            </geometry>
+            <material name="red"/>
+        </visual>
+        <collision>
+            <geometry>
+                <cylinder radius="0.05" length="0.04"/>
+            </geometry>
+        </collision>
+        <xacro:inertial_cylinder mass="0.1" length="0.04" radius="0.05">
+            <origin xyz="0 0 0" rpy="0 0 0"/>
+        </xacro:inertial_cylinder>
     </link>
     <gazebo reference="laser_frame">
@@ -69,4 +58,3 @@
         </sensor>
     </gazebo>
-  </xacro:macro>
 </robot>

File: description/robot.urdf.xacro (robot description, xacro)
@@ -4,3 +4,12 @@
     <xacro:include filename="gazebo_control.xacro"/>
     <xacro:include filename="lidar.xacro" />
+    <!-- Instantiate the RPLIDAR A1, attached to chassis link.
+         Origin is relative to the chassis link frame.
+         Chassis box spans x: 0→0.3, y: -0.15→0.15, z: 0→0.15
+         from chassis link origin (rear-bottom corner).
+         Placing lidar centered on top surface: x=0.15, y=0, z=0.18
+         (z = chassis top 0.15 + half lidar height 0.03) -->
+    <xacro:rplidar_a1 parent="chassis">
+        <origin xyz="0.15 0 0.18" rpy="0 0 0"/>
+    </xacro:rplidar_a1>
 </robot>
