Commit message: simplified launch structure and added dedicated launch files for each sub-system (simulation only).

File: description/gazebo_control.xacro (robot description, xacro)
@@ -1,27 +1,29 @@
 <?xml version="1.0"?>
 <robot xmlns:xacro="http://www.ros.org/wiki/xacro">
-    <gazebo>
-        <plugin name="gz::sim::systems::DiffDrive" filename="gz-sim-diff-drive-system">
-            <!-- Wheel Information -->
-            <left_joint>left_wheel_joint</left_joint>
-            <right_joint>right_wheel_joint</right_joint>
-            <wheel_separation>0.35</wheel_separation>
-            <wheel_radius>0.05</wheel_radius>
-            <!-- Input -->
-            <!-- Use stamped topic for Jazzy compatibility -->
-            <topic>/cmd_vel</topic>
-            <use_stamped_cmd_vel>true</use_stamped_cmd_vel>
-            <!-- Output -->
-            <frame_id>odom</frame_id>
-            <child_frame_id>base_link</child_frame_id>
-            <odom_topic>/odom</odom_topic>
-            <tf_topic>/tf</tf_topic>
-            <odom_publish_frequency>50</odom_publish_frequency>
-        </plugin>
-        <plugin name="gz::sim::systems::JointStatePublisher" filename="gz-sim-joint-state-publisher-system">
-            <topic>/joint_states</topic>
-            <joint_name>left_wheel_joint</joint_name>
-            <joint_name>right_wheel_joint</joint_name>
-        </plugin>
-    </gazebo>
+    <xacro:macro name="gazebo_diff_drive" params="">
+        <gazebo>
+            <plugin name="gz::sim::systems::DiffDrive" filename="gz-sim-diff-drive-system">
+                <!-- Wheel Information -->
+                <left_joint>left_wheel_joint</left_joint>
+                <right_joint>right_wheel_joint</right_joint>
+                <wheel_separation>0.35</wheel_separation>
+                <wheel_radius>0.05</wheel_radius>
+                <!-- Input -->
+                <!-- Use stamped topic for Jazzy compatibility -->
+                <topic>/cmd_vel</topic>
+                <use_stamped_cmd_vel>false</use_stamped_cmd_vel>
+                <!-- Output -->
+                <frame_id>odom</frame_id>
+                <child_frame_id>base_link</child_frame_id>
+                <odom_topic>/odom</odom_topic>
+                <tf_topic>/tf</tf_topic>
+                <odom_publish_frequency>50</odom_publish_frequency>
+            </plugin>
+            <plugin name="gz::sim::systems::JointStatePublisher" filename="gz-sim-joint-state-publisher-system">
+                <topic>/joint_states</topic>
+                <joint_name>left_wheel_joint</joint_name>
+                <joint_name>right_wheel_joint</joint_name>
+            </plugin>
+        </gazebo>
+    </xacro:macro>
 </robot>

File: description/lidar.xacro (robot description, xacro)
@@ -2,5 +2,5 @@
 <robot xmlns:xacro="http://www.ros.org/wiki/xacro">
   <!-- Macro parameters: parent link, XYZ offset, RPY offset -->
-  <xacro:macro name="rplidar_a1" params="parent *origin">
+  <xacro:macro name="rplidar_a1" params="parent use_sim:=false *origin">
     <joint name="laser_joint" type="fixed">
       <xacro:insert_block name="origin"/>
@@ -33,40 +33,42 @@
       </inertial>
     </link>
-    <gazebo reference="laser_frame">
-        <sensor name="laser" type="gpu_lidar">
-            <pose> 0 0 0 0 0 0 </pose>
-            <topic>/scan</topic>
-            <gz_frame_id>laser_frame</gz_frame_id>
-            <update_rate>5</update_rate>
-            <ray>
-                <scan>
-                    <horizontal>
-                        <samples>360</samples>
-                        <resolution>1</resolution>
-                        <min_angle>-3.14159</min_angle>
-                        <max_angle>3.14159</max_angle>
-                    </horizontal>
-                    <vertical>
-                        <samples>1</samples>
-                        <resolution>0.1</resolution>
-                        <min_angle>0</min_angle>
-                        <max_angle>0</max_angle>
-                    </vertical>
-                </scan>
-                <range>
-                    <min>0.15</min>
-                    <max>12.0</max>
-                    <resolution>0.01</resolution>
-                </range>
-                <noise>
-                    <type>gaussian</type>
-                    <mean>0.0</mean>
-                    <stddev>0.01</stddev>
-                </noise>
-            </ray>
-            <always_on>1</always_on>
-            <visualize>true</visualize>
-        </sensor>
-    </gazebo>
+    <xacro:if value="${use_sim}">
+      <gazebo reference="laser_frame">
+          <sensor name="laser" type="gpu_lidar">
+              <pose> 0 0 0 0 0 0 </pose>
+              <topic>/scan</topic>
+              <gz_frame_id>laser_frame</gz_frame_id>
+              <update_rate>5</update_rate>
+              <ray>
+                  <scan>
+                      <horizontal>
+                          <samples>360</samples>
+                          <resolution>1</resolution>
+                          <min_angle>-3.14159</min_angle>
+                          <max_angle>3.14159</max_angle>
+                      </horizontal>
+                      <vertical>
+                          <samples>1</samples>
+                          <resolution>0.1</resolution>
+                          <min_angle>0</min_angle>
+                          <max_angle>0</max_angle>
+                      </vertical>
+                  </scan>
+                  <range>
+                      <min>0.15</min>
+                      <max>12.0</max>
+                      <resolution>0.01</resolution>
+                  </range>
+                  <noise>
+                      <type>gaussian</type>
+                      <mean>0.0</mean>
+                      <stddev>0.01</stddev>
+                  </noise>
+              </ray>
+              <always_on>1</always_on>
+              <visualize>true</visualize>
+          </sensor>
+      </gazebo>
+    </xacro:if>
   </xacro:macro>
 </robot>

File: description/robot.urdf.xacro (robot description, xacro)
@@ -1,8 +1,28 @@
 <?xml version="1.0"?>
 <robot xmlns:xacro="http://www.ros.org/wiki/xacro"  name="robot">
+    <xacro:arg name="use_sim" default="false" />
+    <xacro:arg name="use_lidar" default="false" />
+    <xacro:arg name="use_camera" default="false" />
     <xacro:include filename="robot_core.xacro" />
     <xacro:include filename="gazebo_control.xacro"/>
     <xacro:include filename="lidar.xacro" />
     <xacro:include filename="camera.xacro" />
+    <!-- Gazebo drive + joint-state plugins -->
+    <xacro:if value="$(arg use_sim)">
+        <xacro:gazebo_diff_drive/>
+    </xacro:if>
+    <!-- Optional lidar -->
+    <xacro:if value="$(arg use_lidar)">
+        <xacro:rplidar_a1 parent="chassis" use_sim="$(arg use_sim)">
+        <origin xyz="0.15 0 0.18" rpy="0 0 0"/>
+        </xacro:rplidar_a1>
+    </xacro:if>
+    <!-- Optional camera -->
+    <xacro:if value="$(arg use_camera)">
+        <xacro:pi_camera_v2 parent="chassis" use_sim="$(arg use_sim)">
+        <origin xyz="0.300 0.0 0.075" rpy="0 0 0"/>
+        </xacro:pi_camera_v2>
+    </xacro:if>
+    <!-- Commented out the below on 3/23/26 -->
     <!-- Instantiate the RPLIDAR A1, attached to chassis link.
          Origin is relative to the chassis link frame.
@@ -11,7 +31,9 @@
          Placing lidar centered on top surface: x=0.15, y=0, z=0.18
          (z = chassis top 0.15 + half lidar height 0.03) -->
+    <!--
     <xacro:rplidar_a1 parent="chassis">
         <origin xyz="0.15 0 0.18" rpy="0 0 0"/>
     </xacro:rplidar_a1>
+    -->
     <!--
         NOTE: The camera link/joint are defined entirely within camera.xacro
