Commit message: updated robot urdf to reflect v2 geometry.

File: description/gazebo_control.xacro (robot description, xacro)
@@ -7,6 +7,6 @@
                 <left_joint>left_wheel_joint</left_joint>
                 <right_joint>right_wheel_joint</right_joint>
-                <wheel_separation>0.35</wheel_separation>
-                <wheel_radius>0.05</wheel_radius>
+                <wheel_separation>0.298</wheel_separation>
+                <wheel_radius>0.034</wheel_radius>
                 <!-- Input -->
                 <!-- Use stamped topic for Jazzy compatibility -->

File: description/lidar.xacro (robot description, xacro)
@@ -11,6 +11,6 @@
       <visual>
         <geometry>
-          <!-- A1 approximate dimensions: 98.5mm diameter, 60mm height -->
-          <cylinder radius="0.0493" length="0.060"/>
+          <!-- A1 approximate dimensions: 70mm diameter, 54.5mm height -->
+          <cylinder radius="0.035" length="0.0545"/>
         </geometry>
         <material name="lidar_red">
@@ -20,11 +20,12 @@
       <collision>
         <geometry>
-          <cylinder radius="0.0493" length="0.060"/>
+          <cylinder radius="0.035" length="0.0545"/>
         </geometry>
       </collision>
+      <!--
       <inertial>
-        <!-- RPLIDAR A1M8 mass: ~170g -->
+        <! RPLIDAR A1M8 mass: ~170g >
         <mass value="0.170"/>
-        <!-- Solid cylinder: Ixx = Iyy = m(3r² + h²)/12, Izz = mr²/2 -->
+        <! Solid cylinder: Ixx = Iyy = m(3r² + h²)/12, Izz = mr²/2 >
         <inertia
           ixx="0.000214" ixy="0.0" ixz="0.0"
@@ -32,4 +33,8 @@
           izz="0.000205"/>
       </inertial>
+      -->
+      <xacro:inertial_cylinder mass="0.170" length="0.0545" radius="0.035">
+        <origin xyz="0 0 0" rpy="0 0 0"/>
+      </xacro:inertial_cylinder>
     </link>
     <xacro:if value="${use_sim}">

File: description/robot.urdf.xacro (robot description, xacro)
@@ -15,5 +15,5 @@
     <xacro:if value="$(arg use_lidar)">
         <xacro:rplidar_a1 parent="chassis" use_sim="$(arg use_sim)">
-        <origin xyz="0.15 0 0.18" rpy="0 0 0"/>
+            <origin xyz="0.09 0.0 0.13575" rpy="0 0 0"/>
         </xacro:rplidar_a1>
     </xacro:if>
@@ -21,5 +21,5 @@
     <xacro:if value="$(arg use_camera)">
         <xacro:pi_camera_v2 parent="chassis" use_sim="$(arg use_sim)">
-        <origin xyz="0.300 0.0 0.075" rpy="0 0 0"/>
+            <origin xyz="0.10325 -0.115 0.1235" rpy="0 0 0"/>
         </xacro:pi_camera_v2>
     </xacro:if>

File: description/robot_core.xacro (robot description, xacro)
@@ -28,18 +28,18 @@
     <link name="chassis">
         <visual>
-            <origin xyz="0.14 0 0.05" rpy="0 0 0"/>
+            <origin xyz="0.09 0 0.0635" rpy="0 0 0"/>
             <geometry>
-                <box size="0.28 0.26 0.10"/>
+                <box size="0.28 0.26 0.09"/>
             </geometry>
             <material name="white"/>
         </visual>
         <collision>
-            <origin xyz="0.14 0 0.05" rpy="0 0 0"/>
+            <origin xyz="0.09 0 0.0635" rpy="0 0 0"/>
             <geometry>
-                <box size="0.28 0.26 0.10"/>
+                <box size="0.28 0.26 0.09"/>
             </geometry>
         </collision>
-        <xacro:inertial_box mass="0.5" x="0.28" y="0.26" z="0.10">
-            <origin xyz="0.14 0 0.05" rpy="0 0 0"/>
+        <xacro:inertial_box mass="0.5" x="0.28" y="0.26" z="0.09">
+            <origin xyz="0.09 0 0.0635" rpy="0 0 0"/>
         </xacro:inertial_box>
     </link>
@@ -50,5 +50,5 @@
         <origin xyz="0 0.149 0" rpy="-${pi/2} 0 0"/>
         <axis xyz="0 0 1"/>
-        <limit effort="0.05" velocity="10.0"/>
+        <limit effort="1.0" velocity="10.0"/>
     </joint>
     <link name="left_wheel">
@@ -74,5 +74,5 @@
         <origin xyz="0 -0.149 0" rpy="${pi/2} 0 0"/>
         <axis xyz="0 0 -1"/>
-        <limit effort="0.05" velocity="10.0"/>
+        <limit effort="1.0" velocity="10.0"/>
     </joint>
     <link name="right_wheel">
@@ -96,10 +96,10 @@
         <parent link="chassis"/>
         <child link="caster_wheel"/>
-        <origin xyz="0.18 0 0" rpy="0 0 0"/>
+        <origin xyz="0.18 0 0.0185" rpy="0 0 0"/> <!-- "0.09 0 -0.045" -->
     </joint>
     <link name="caster_wheel">
         <visual>
             <geometry>
-                <sphere radius="0.034" />
+                <sphere radius="0.0525" />
             </geometry>
             <material name="black"/>
@@ -107,8 +107,8 @@
         <collision>
             <geometry>
-                <sphere radius="0.034" />
+                <sphere radius="0.0525" />
             </geometry>
         </collision>
-        <xacro:inertial_sphere mass="0.1" radius="0.034">
+        <xacro:inertial_sphere mass="0.1" radius="0.0525">
             <origin xyz="0 0 0" rpy="0 0 0"/>
         </xacro:inertial_sphere>
